Commit message: changed order of urdf elements and added mujoco files

File: robotmodels/dingo_kinova/urdf/dingo_kinova_gripper.urdf (robot description, URDF)
Before this commit: robot dingo_kinova, 31 links, 30 joints
Links:
- link arm_gripper_base_link: geometry collision mesh filename=../meshes/kinova/gripper_base_link.STL; visual mesh filename=../meshes/kinova/gripper_base_link.STL
